Commit message: update for sensorlib

File: xil_carma_training/cdasim_config/carma_training/vehicle/calibration/urdf/carma.urdf (robot description, URDF)
Before this commit: robot vehicle_platform, 13 links, 12 joints
Links:
- removed link gps
- removed link host_vehicle
- removed link mobileye
- removed link ned_heading
- removed link novatel_imu
- removed link radar_fc
- removed link radar_fl
- removed link radar_fr
- removed link radar_rl
- removed link radar_rr
- removed link vehicle_front
- removed link velodyne
- added link pinpoint
- link base_link: geometry 
Joints:
- removed joint base_link_to_host_vehicle
- removed joint base_link_to_novatel
- removed joint base_link_to_novatel_imu
- removed joint base_link_to_vehicle_front
- removed joint gnss_to_ned_heading
- removed joint lidar
- removed joint mobileye
- removed joint radar_fc
- removed joint radar_fl
- removed joint radar_fr
- removed joint radar_rl
- removed joint radar_rr
- added joint pinpoint: type fixed, parent base_link, child pinpoint, origin xyz=0 0 0 rpy=3.145159 0 0
